File: Motherboard_V2.kicad_sch (KiCad schematic)
At the start: 30 parts, among them J1 GSB1C41110SSHR, J2 S2B-PH-K-SLFSN, J3 B8B-PH-K-SLFSN, J4 Conn_02x04_Counter_Clockwise, Q1 AONR21307, U3 LM2596S-5, U4 LM2596S-12

Commit message: Assign footprints to U2 (ESP32-C6), L1 (33uH), and L2 (68uH)
- Copy ESP32-C6.pretty footprint from Control Board project for U2
- Add Bourns SRN6045 footprint for L1 (33uH) to SWM.pretty
- Add Bourns SRR1210 footprint for L2 (68uH) to SWM.pretty
- Register ESP32-C6 footprint library in fp-lib-table
- Update schematic footprint assignments for all three components

Co-Authored-By: Claude Opus 4.5 <noreply@anthropic.com>
Parts:
- L1: footprint (none) -> SWM:IND_BOURNS_SRN6045
- L2: footprint (none) -> SWM:IND_BOURNS_SRR1210
- U2: footprint (none) -> ESP32-C6:E
Changed lines of the file:
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@@
 			)
 		)
-		(property "Footprint" ""
+		(property "Footprint" "ESP32-C6:E"
 			(at 194.31 44.45 0)
 			(effects
@@
 			)
 		)
-		(property "Footprint" ""
+		(property "Footprint" "SWM:IND_BOURNS_SRN6045"
 			(at 129.54 87.63 0)
 			(effects
@@
 			)
 		)
-		(property "Footprint" ""
+		(property "Footprint" "SWM:IND_BOURNS_SRR1210"
 			(at 129.54 62.23 0)
 			(effects

Commit message: Bundle HUSB238A_002D footprint locally for U1
Copy footprint from KiCad's Package_DFN_QFN library into SWM.pretty
so the project doesn't depend on a specific KiCad version having it.

Co-Authored-By: Claude Opus 4.5 <noreply@anthropic.com>
Parts:
- U1: footprint Package_DFN_QFN:HUSB238A_002D -> SWM:HUSB238A_002D
Changed lines of the file:
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@@
 			)
 		)
-		(property "Footprint" "Package_DFN_QFN:HUSB238A_002D"
+		(property "Footprint" "SWM:HUSB238A_002D"
 			(at 57.15 156.21 0)
 			(effects

Commit message: Add USB-C footprints and update PCB layout
- Add CONN12_C-31-M-12_HRO and USB_C_Receptacle_HRO_TYPE-C-31-M-12 footprints
- Update PCB layout with component placement and routing
- Add new component symbols to SWM Components library
- Update schematic with design changes
- Register new footprint and symbol libraries in library tables

Co-Authored-By: Claude Opus 4.6 <noreply@anthropic.com>
Parts:
- removed J1: GSB1C41110SSHR, SWM:AMPHENOL_GSB1C41110SSHR, symbol GSB1C41110SSHR:GSB1C41110SSHR
- added J1: TYPE-C-31-M-12, SWM:CONN12_C-31-M-12_HRO, symbol 2026-02-02_06-36-16:TYPE-C-31-M-12
Connections:
- net CC1: now also J1.A5
- net CC2: now also J1.B5
- net D+: now also J1.A6, J1.A7
- net D-: now also J1.B6, J1.B7
- net GND: now also R6.2, J1.13, J1.14, J1.15, J1.16, J1.A1-B12, J1.B1-A12
- net USB_GATE: now also Q1.4; no longer U1.10 (GATE)
- net VBUS: now also J1.A4-B9, J1.B4-A9
- net V_BATT_SENSE: now also C10.2
- net at R3.1: now also U1.10 (GATE); no longer Q1.4
Other:
- moved on the sheet: C10, R3
